File: hardware/pcb/RF Amplifier.kicad_sch (KiCad schematic)
At the start: 25 parts, among them J401 BNC_Rosenberger, SW401 Gain Select, U401 OPA690

Commit message: Update all repo links after moving the repo to the Domesday86 github organisation
Other:
- company: https://github.com/simoninns/DomesdayDuplicator -> https://github.com/Domesday86/DomesdayDuplicator
Changed lines of the file:
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@@
 		(date "2026-08-13")
 		(rev "3.0.2")
-		(company "https://github.com/simoninns/DomesdayDuplicator")
+		(company "https://github.com/Domesday86/DomesdayDuplicator")
 		(comment 1 "(c)2018-2026 Simon Inns")
 		(comment 2 "License: Attribution-ShareAlike 4.0 International (CC BY-SA 4.0)")
